File: Midi_Controller_02/Midi_Controller_02.kicad_pcb (KiCad board)
At the start: 2 copper layers, 254.1 x 134.1 mm, 150 parts, among them J4 COL HEADER, J5 CA HEADER

Commit message: initial commit
Parts:
- added REF**: MountingHole_2.2mm_M2, MountingHole:MountingHole_2.2mm_M2, F.Cu at (4.00, 131.0)
- added REF**: MountingHole_2.2mm_M2, MountingHole:MountingHole_2.2mm_M2, F.Cu at (250.0, 131.0)
- added REF**: MountingHole_2.2mm_M2, MountingHole:MountingHole_2.2mm_M2, F.Cu at (250.0, 4.00)
- moved J4 163.0 mm to (145.1, 131.7), turned to 90 degrees
- moved J5 16.5 mm to (144.7, 4.83)
Routing:
- net /CONTROLLER-MATRIX/CB8: track 162.7 -> 385.8 mm, vias 8 -> 19
- net /CONTROLLER-MATRIX/COL0: track 140.7 -> 275.3 mm
- net /CONTROLLER-MATRIX/CA1: track 229.5 -> 363.2 mm, vias 0 -> 2
- net /CONTROLLER-MATRIX/CA8: track 229.0 -> 357.5 mm, vias 12 -> 20
- net /CONTROLLER-MATRIX/CA7: track 253.9 -> 380.6 mm, vias 12 -> 16
- net /CONTROLLER-MATRIX/CA2: track 262.6 -> 383.7 mm, vias 6 -> 8
- net /CONTROLLER-MATRIX/COL5: track 85.7 -> 204.3 mm, vias 6 -> 10
- net /CONTROLLER-MATRIX/COL1: track 133.8 -> 251.5 mm
- net /CONTROLLER-MATRIX/COL2: track 123.0 -> 231.2 mm, vias 6 -> 7
- net /CONTROLLER-MATRIX/CB9: track 107.9 -> 208.4 mm, vias 0 -> 1
- net /CONTROLLER-MATRIX/COL4: track 111.6 -> 210.8 mm, vias 6 -> 9
- net /CONTROLLER-MATRIX/CA5: track 248.9 -> 347.6 mm, vias 6 -> 8
- net /CONTROLLER-MATRIX/COL3: track 128.7 -> 218.5 mm
- net /CONTROLLER-MATRIX/COL15: track 109.9 -> 197.4 mm
- net /CONTROLLER-MATRIX/CA6: track 268.7 -> 352.4 mm, vias 11 -> 13
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Other:
- board size 254.1 x 134.1 mm -> 254 x 135 mm
