File: Midi_Controller_02/Midi_Controller_02_Cntrol/Midi_Controller_02_Cntrol.kicad_pcb (KiCad board)
At the start: 2 copper layers, 110 x 55 mm, 50 parts, among them J1 ISP Header, J2 UJ20-C-H-G-SMT-1-P16-TR, J3 ISP Header, J4 COL HEADER, J5 CA HEADER, SW1 SW_Push, U1 ATmega328P-M, U2 74154, U3 IS31FL3731-SA, U4 ATmega16U2-A, U5 AMS1117-3.3, Y1 16MHz, Y2 16MHz

Commit message: initial commit
Parts:
- added REF**: MountingHole_2.2mm_M2, MountingHole:MountingHole_2.2mm_M2, F.Cu at (4.00, 4.00)
- added REF**: MountingHole_2.2mm_M2, MountingHole:MountingHole_2.2mm_M2, F.Cu at (5.00, 51.0)
- added REF**: MountingHole_2.2mm_M2, MountingHole:MountingHole_2.2mm_M2, F.Cu at (106.0, 4.00)
- added REF**: MountingHole_2.2mm_M2, MountingHole:MountingHole_2.2mm_M2, F.Cu at (106.0, 51.0)
- J5: footprint Connector_PinHeader_2.54mm:PinHeader_2x08_P2.54mm_Horizontal -> Connector_PinHeader_2.54mm:PinHeader_2x09_P2.54mm_Horizontal
- moved C8 77.8 mm to (73.5, 30.9), turned to 180 degrees
- moved TP1 30.8 mm to (63.4, 3.95)
- moved TP2 22.4 mm to (68.1, 4.06)
- moved R1 16.6 mm to (74.4, 5.95), turned to -90 degrees
- moved R2 13.5 mm to (76.9, 6.05), turned to -90 degrees
- moved J5 6.01 mm to (84.9, 4.90), turned to 0 degrees
- moved TP6 1.84 mm to (71.7, 7.47)
- moved R4 1.69 mm to (67.0, 16.8)
- moved R5 1.69 mm to (67.0, 19.5)
Routing:
- net /CB8: track 58.4 -> 15.6 mm
- net /CB7: track 58.9 -> 21.3 mm
- net /CB6: track 52.7 -> 18.7 mm
- net /CB5: track 53.2 -> 23.0 mm
- net /CB4: track 47.1 -> 21.2 mm
- net /CB2: track 39.9 -> 15.2 mm, vias 0 -> 1
- net /CB3: track 47.6 -> 25.5 mm
- net /CB1: track 36.3 -> 18.0 mm, vias 0 -> 1
- net /COL15: track 8.56 -> 24.6 mm
- net /I2S_SCL: track 58.0 -> 70.4 mm
- net /COL11: track 24.5 -> 14.2 mm
- net /COL1: track 21.3 -> 31.3 mm
- net /COL7: track 29.0 -> 39.0 mm
- net /CA2: track 12.2 -> 22.0 mm
- net /COL3: track 22.6 -> 32.5 mm
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