File: Midi_Controller_02/Midi_Controller_02_Cntrol/Midi_Controller_02_Cntrol.kicad_sch (KiCad schematic)
At the start: 50 parts, among them J1 ISP Header, J2 UJ20-C-H-G-SMT-1-P16-TR, J3 ISP Header, J4 COL HEADER, J5 CA HEADER, SW1 SW_Push, U1 ATmega328P-M, U2 74154, U3 IS31FL3731-SA, U4 ATmega16U2-A, U5 AMS1117-3.3, Y1 16MHz, Y2 16MHz

Commit message: initial commit
Parts:
- C17: value 20uF -> 22uF
Other:
- moved on the sheet: C16, C17, TP9, U5
